File: hw/LT1161_2.sch (KiCad schematic (older format))
At the start: 9 parts, among them U401 MOSFET_DRIVER_LT1161, U402 MOSFET_IPG20N04S4L11ATMA1, U403 MOSFET_IPG20N04S4L11ATMA1, U404 MOSFET_DRIVER_MCP1402T-E/OT

Commit message: creating hw 3.0.0
Parts:
- added C403, C404: 100nF, kemet:0603, symbol 100nF
- added U?: MOSFET_IPG20N04S4L11ATMA1, usevolt:PG-TDSON-8-4, symbol MOSFET_IPG20N04S4L11ATMA1
Connections:
- net GND: now also C403.1 (C1), C404.1 (C1)
- net OUT+: now also U?.1 (S1), U?.3 (S2)
- net Sheet59847684/SENSE-: now also U401.15 (SENSE3), U402.6 (D2)
- net Sheet5989C9E5/SENSE-: now also U401.13 (SENSE4), U?.2 (G1), U?.6 (D2); no longer U402.6 (D2)
- net at C401.1 (C1), C402.1 (C1), D401.P$2 (N)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: no longer U401.13 (SENSE4), U401.15 (SENSE3)
- net at U401.12 (GATE4): now also U?.4 (G2), U?.5 (D1); no longer U402.4 (G2)
- net at U401.14 (GATE3), U402.2 (G1): now also U402.4 (G2)
- net at U401.6 (TIMER3): now also C403.2 (C2)
- net at U401.8 (TIMER4): now also C404.2 (C2)
Other:
- moved on the sheet: R401A, R401B, R401C, R401D, U402
