File: hw/currentSense.sch (KiCad schematic (older format))
At the start: 2 parts, among them U501 ZXCT1086

Commit message: creating hw 3.0.0
Changed lines of the file:
@@
 $Descr A4 11693 8268
 encoding utf-8
-Sheet 5 11
+Sheet 5 10
 Title "MSB current sense sheet"
 Date "2017-02-05"
@@
 AR Path="/598914ED/58BE8E88/594D8B7D" Ref="U1001"  Part="1"
 AR Path="/598914ED/58BE8E96/594D8B7D" Ref="U1101"  Part="1"
-F 0 "U801" H 5425 3887 60  0000 C CNN
+F 0 "U501" H 5425 3887 60  0000 C CNN
 F 1 "ZXCT1086" H 5425 3781 60  0000 C CNN
 F 2 "usevolt:SOT-25" H 5100 4050 60  0001 C CNN
@@
 $EndComp
 $Comp
-L GND #PWR034
+L GND #PWR502
 U 1 1 594D8B7E
 P 5050 4000
-AR Path="/59891726/59847685/594D8B7E" Ref="#PWR034"  Part="1"
-AR Path="/59891726/5989C9E6/594D8B7E" Ref="#PWR036"  Part="1"
+AR Path="/59891726/59847685/594D8B7E" Ref="#PWR502"  Part="1"
+AR Path="/59891726/5989C9E6/594D8B7E" Ref="#PWR602"  Part="1"
 AR Path="/598914ED/595CED4D/594D8B7E" Ref="#PWR042"  Part="1"
 AR Path="/598914ED/58BE8E7A/594D8B7E" Ref="#PWR044"  Part="1"
 AR Path="/598914ED/58BE8E88/594D8B7E" Ref="#PWR046"  Part="1"
 AR Path="/598914ED/58BE8E96/594D8B7E" Ref="#PWR048"  Part="1"
-F 0 "#PWR048" H 5050 3750 50  0001 C CNN
+F 0 "#PWR502" H 5050 3750 50  0001 C CNN
 F 1 "GND" H 5055 3827 50  0000 C CNN
 F 2 "" H 5050 4000 50  0000 C CNN
@@
 $EndComp
 $Comp
-L +3V3 #PWR035
+L +3V3 #PWR501
 U 1 1 589841AE
 P 5050 3350
-AR Path="/59891726/59847685/589841AE" Ref="#PWR035"  Part="1"
-AR Path="/59891726/5989C9E6/589841AE" Ref="#PWR037"  Part="1"
+AR Path="/59891726/59847685/589841AE" Ref="#PWR501"  Part="1"
+AR Path="/59891726/5989C9E6/589841AE" Ref="#PWR601"  Part="1"
 AR Path="/598914ED/595CED4D/589841AE" Ref="#PWR043"  Part="1"
 AR Path="/598914ED/58BE8E7A/589841AE" Ref="#PWR045"  Part="1"
 AR Path="/598914ED/58BE8E88/589841AE" Ref="#PWR047"  Part="1"
 AR Path="/598914ED/58BE8E96/589841AE" Ref="#PWR049"  Part="1"
-F 0 "#PWR049" H 5050 3200 50  0001 C CNN
+F 0 "#PWR501" H 5050 3200 50  0001 C CNN
 F 1 "+3V3" H 5065 3523 50  0000 C CNN
 F 2 "" H 5050 3350 50  0000 C CNN
@@
 AR Path="/598914ED/58BE8E88/589858BC" Ref="R1001"  Part="1"
 AR Path="/598914ED/58BE8E96/589858BC" Ref="R1101"  Part="1"
-F 0 "R801" V 6208 3508 45  0000 L CNN
+F 0 "R501" V 6208 3508 45  0000 L CNN
 F 1 "LRMAT2512-R002FT4" V 6292 3508 45  0000 L CNN
 F 2 "usevolt:2512" H 6230 3600 20  0001 C CNN
