File: hw/heater.sch (KiCad schematic (older format))
At the start: 6 parts, among them U802 VN5E010AH, U803 VN5E010AH

Commit message: hw 2.2 ordered from seeed
Parts:
- added D801: SCHOTTKY_DIODE_V40PW10C, usevolt:SlimDPAK, symbol SCHOTTKY_DIODE_V40PW10C
Connections:
- wire segments 33 -> 37
Changed lines of the file:
@@
 	5500 5000 5500 3950
 Connection ~ 5500 3950
-Wire Wire Line
-	7050 4900 7050 3700
 Connection ~ 7050 3700
 Wire Wire Line
@@
 	1    0    0    -1
 $EndComp
+Wire Wire Line
+	7050 4900 7050 3700
+$Comp
+L SCHOTTKY_DIODE_V40PW10C D801
+U 1 1 5A394B01
+P 7700 4450
+F 0 "D801" H 7700 4797 60  0000 C CNN
+F 1 "SCHOTTKY_DIODE_V40PW10C" H 7700 4691 60  0000 C CNN
+F 2 "usevolt:SlimDPAK" H 7500 4100 60  0001 C CNN
+F 3 "http://www.farnell.com/datasheets/2245239.pdf?_ga=2.16591231.874534928.1505194133-1862443086.1504075057" H 7500 4100 60  0001 C CNN
+F 4 "2535169" H 8050 5050 60  0001 C CNN "1st Source Part Number"
+F 5 "Digikey" H 8150 5150 60  0001 C CNN "2nd Source"
+F 6 "Farnell" H 7950 4950 60  0001 C CNN "1st Source"
+F 7 "V40PW10CHM3/I" H 7850 4850 60  0001 C CNN "Manufacturer Part Number"
+F 8 "V40PW10CHM3/IGICT-ND" H 8250 5250 60  0001 C CNN "2nd Source Part Number"
+F 9 "VISHAY" H 7750 4750 60  0001 C CNN "Manufacturer"
+	1    7700 4450
+	-1   0    0    -1
+$EndComp
+Wire Wire Line
+	7300 4400 7050 4400
+Connection ~ 7050 4400
+$Comp
+L GND #PWR807
+U 1 1 5A394BA1
+P 8300 4600
+F 0 "#PWR807" H 8300 4350 50  0001 C CNN
+F 1 "GND" H 8305 4427 50  0000 C CNN
+F 2 "" H 8300 4600 50  0000 C CNN
+F 3 "" H 8300 4600 50  0000 C CNN
+	1    8300 4600
+	1    0    0    -1
+$EndComp
+Wire Wire Line
+	8300 4350 8300 4600
+Wire Wire Line
+	8300 4450 8100 4450
+Wire Wire Line
+	8300 4350 8100 4350
+Connection ~ 8300 4450
 $EndSCHEMATC
